File: RX EQ Shield.sch (KiCad schematic (older format))
At the start: 6 parts

Commit message: Filter calculations, gain stage, oscillation protection
Other:
- note added: "TODO:\n- Filter component calculations"
- note removed: "TODO:\n- All Op-Amps need filtering for feedback\n- Filter component calculations"
Changed lines of the file:
@@
 EQ Channels have 10k output resistors incorporated
 Text Notes 5250 4700 0    50   ~ 0
-TODO:\n- All Op-Amps need filtering for feedback\n- Filter component calculations
+TODO:\n- Filter component calculations
 $Comp
 L Device:R R?

Commit message: WIP
Other:
- note removed: "TODO:\n- Filter component calculations"
Changed lines of the file:
@@
 Text Notes 5000 3950 0    50   ~ 0
 EQ Channels have 10k output resistors incorporated
-Text Notes 5250 4700 0    50   ~ 0
-TODO:\n- Filter component calculations
 $Comp
 L Device:R R?

Commit message: Ferrite beads and annotations
Parts:
- gave numbers to parts that had none: 6
Changed lines of the file:
@@
 $EndSheet
 $Comp
-L power:GNDA #PWR?
+L power:GNDA #PWR04
 U 1 1 5E4114FD
 P 4850 1950
-F 0 "#PWR?" H 4850 1700 50  0001 C CNN
+F 0 "#PWR04" H 4850 1700 50  0001 C CNN
 F 1 "GNDA" H 4855 1777 50  0000 C CNN
 F 2 "" H 4850 1950 50  0001 C CNN
@@
 	5150 2550 5150 1750
 $Comp
-L Connector:Conn_01x02_Female TP?
+L Connector:Conn_01x02_Female TP1
 U 1 1 5E412C7A
 P 5850 950
-F 0 "TP?" H 5878 926 50  0000 L CNN
+F 0 "TP1" H 5878 926 50  0000 L CNN
 F 1 "Conn_01x02_Female" H 5878 835 50  0000 L CNN
 F 2 "" H 5850 950 50  0001 C CNN
@@
 $EndComp
 $Comp
-L power:GNDA #PWR?
+L power:GNDA #PWR01
 U 1 1 5E413291
 P 5400 1050
-F 0 "#PWR?" H 5400 800 50  0001 C CNN
+F 0 "#PWR01" H 5400 800 50  0001 C CNN
 F 1 "GNDA" H 5405 877 50  0000 C CNN
 F 2 "" H 5400 1050 50  0001 C CNN
@@
 $EndSheet
 $Comp
-L Connector_Generic:Conn_02x04_Odd_Even J?
+L Connector_Generic:Conn_02x04_Odd_Even J1
 U 1 1 5E41835B
 P 1450 1350
-F 0 "J?" H 1500 1667 50  0000 C CNN
+F 0 "J1" H 1500 1667 50  0000 C CNN
 F 1 "Conn_02x04_Odd_Even" H 1500 1576 50  0000 C CNN
 F 2 "" H 1450 1350 50  0001 C CNN
@@
 $EndComp
 $Comp
-L power:GND #PWR?
+L power:GND #PWR02
 U 1 1 5E41923D
 P 800 1150
-F 0 "#PWR?" H 800 900 50  0001 C CNN
+F 0 "#PWR02" H 800 900 50  0001 C CNN
 F 1 "GND" H 805 977 50  0000 C CNN
 F 2 "" H 800 1150 50  0001 C CNN
@@
 $EndComp
 $Comp
-L power:+5V #PWR?
+L power:+5V #PWR03
 U 1 1 5E419402
 P 2050 1250
-F 0 "#PWR?" H 2050 1100 50  0001 C CNN
+F 0 "#PWR03" H 2050 1100 50  0001 C CNN
 F 1 "+5V" H 2065 1423 50  0000 C CNN
 F 2 "" H 2050 1250 50  0001 C CNN
@@
 	3300 1650 3750 1650
 $Comp
-L power:+5V #PWR?
+L power:+5V #PWR05
 U 1 1 5E457588
 P 1700 2850
-F 0 "#PWR?" H 1700 2700 50  0001 C CNN
+F 0 "#PWR05" H 1700 2700 50  0001 C CNN
 F 1 "+5V" H 1715 3023 50  0000 C CNN
 F 2 "" H 1700 2850 50  0001 C CNN
@@
 $EndComp
 $Comp
-L power:GND #PWR?
+L power:GND #PWR06
 U 1 1 5E4577BE
 P 1700 3550
-F 0 "#PWR?" H 1700 3300 50  0001 C CNN
+F 0 "#PWR06" H 1700 3300 50  0001 C CNN
 F 1 "GND" H 1705 3377 50  0000 C CNN
 F 2 "" H 1700 3550 50  0001 C CNN
@@
 $EndComp
 $Comp
-L Device:C C?
+L Device:C C1
 U 1 1 5E457AED
 P 1700 3200
-F 0 "C?" H 1815 3246 50  0000 L CNN
+F 0 "C1" H 1815 3246 50  0000 L CNN
 F 1 "10uF" H 1815 3155 50  0000 L CNN
 F 2 "" H 1738 3050 50  0001 C CNN
@@
 Bulk Decoupling
 $Comp
-L Device:C C?
+L Device:C C2
 U 1 1 5E459F4F
 P 2150 3200
-F 0 "C?" H 2265 3246 50  0000 L CNN
+F 0 "C2" H 2265 3246 50  0000 L CNN
 F 1 "1uF" H 2265 3155 50  0000 L CNN
 F 2 "" H 2188 3050 50  0001 C CNN
@@
 EQ Channels have 10k output resistors incorporated
 $Comp
-L Device:R R?
+L Device:R R1
 U 1 1 5E4AE546
 P 8400 2250
-F 0 "R?" V 8193 2250 50  0000 C CNN
+F 0 "R1" V 8193 2250 50  0000 C CNN
 F 1 "1" V 8284 2250 50  0000 C CNN
 F 2 "" V 8330 2250 50  0001 C CNN
@@
 $EndComp
 $Comp
-L Device:R R?
+L Device:R R2
 U 1 1 5E4AE6C0
 P 8400 2500
-F 0 "R?" V 8193 2500 50  0000 C CNN
+F 0 "R2" V 8193 2500 50  0000 C CNN
 F 1 "1" V 8284 2500 50  0000 C CNN
 F 2 "" V 8330 2500 50  0001 C CNN

Commit message: Layout, 2020-05 order
Parts:
- removed TP1: Conn_01x02_Female, symbol Connector:Conn_01x02_Female
- C1, C2: footprint (none) -> Capacitors_SMD:C_0805_HandSoldering
- J1: footprint (none) -> Pin_Headers:Pin_Header_Straight_2x04_Pitch2.54mm
- R1, R2: footprint (none) -> Resistors_SMD:R_0805_HandSoldering
Connections:
- net +5V: now also J1.7 (Pin_7); no longer J1.2 (Pin_2)
- net Audio_In_L: now also J1.3 (Pin_3); no longer J1.5 (Pin_5)
- net Audio_Out_L: now also J1.4 (Pin_4); no longer J1.6 (Pin_6)
- net Audio_Out_R: now also J1.6 (Pin_6); no longer J1.4 (Pin_4)
- net GND: now also J1.8 (Pin_8); no longer J1.1 (Pin_1)
- net Mic_In: now also J1.1 (Pin_1), J1.2 (Pin_2); no longer J1.7 (Pin_7), J1.8 (Pin_8)
Other:
- note added: "Microphone signal is unmodified \nin this version of the design"
- note removed: "CHECK THIS BEFORE SUBMITTING PCB\n"
- note removed: "Microphone signal is unmodified in this version of the design"
Changed lines of the file:
@@
 Wire Wire Line
 	4850 1900 4850 1950
-Wire Wire Line
-	4450 1750 5100 1750
 $Sheet
 S 5550 2400 750  500
@@
 Wire Wire Line
 	5150 2550 5150 1750
-$Comp
-L Connector:Conn_01x02_Female TP1
-U 1 1 5E412C7A
-P 5850 950
-F 0 "TP1" H 5878 926 50  0000 L CNN
-F 1 "Conn_01x02_Female" H 5878 835 50  0000 L CNN
-F 2 "" H 5850 950 50  0001 C CNN
-F 3 "~" H 5850 950 50  0001 C CNN
-	1    5850 950
-	1    0    0    -1
-$EndComp
-$Comp
-L power:GNDA #PWR01
-U 1 1 5E413291
-P 5400 1050
-F 0 "#PWR01" H 5400 800 50  0001 C CNN
-F 1 "GNDA" H 5405 877 50  0000 C CNN
-F 2 "" H 5400 1050 50  0001 C CNN
-F 3 "" H 5400 1050 50  0001 C CNN
-	1    5400 1050
-	1    0    0    -1
-$EndComp
-Wire Wire Line
-	5400 1050 5650 1050
-Wire Wire Line
-	5650 950  5100 950
-Wire Wire Line
-	5100 950  5100 1750
-Connection ~ 5100 1750
-Wire Wire Line
-	5100 1750 5150 1750
 $Sheet
 S 7000 2150 800  500
@@
 F 0 "J1" H 1500 1667 50  0000 C CNN
 F 1 "Conn_02x04_Odd_Even" H 1500 1576 50  0000 C CNN
-F 2 "" H 1450 1350 50  0001 C CNN
+F 2 "Pin_Headers:Pin_Header_Straight_2x04_Pitch2.54mm" H 1450 1350 50  0001 C CNN
 F 3 "~" H 1450 1350 50  0001 C CNN
 	1    1450 1350
@@
 L power:GND #PWR02
 U 1 1 5E41923D
-P 800 1150
-F 0 "#PWR02" H 800 900 50  0001 C CNN
-F 1 "GND" H 805 977 50  0000 C CNN
-F 2 "" H 800 1150 50  0001 C CNN
-F 3 "" H 800 1150 50  0001 C CNN
-	1    800  1150
+P 1900 1550
+F 0 "#PWR02" H 1900 1300 50  0001 C CNN
+F 1 "GND" H 1905 1377 50  0000 C CNN
+F 2 "" H 1900 1550 50  0001 C CNN
+F 3 "" H 1900 1550 50  0001 C CNN
+	1    1900 1550
 	1    0    0    -1
 $EndComp
@@
 L power:+5V #PWR03
 U 1 1 5E419402
-P 2050 1250
-F 0 "#PWR03" H 2050 1100 50  0001 C CNN
-F 1 "+5V" H 2065 1423 50  0000 C CNN
-F 2 "" H 2050 1250 50  0001 C CNN
-F 3 "" H 2050 1250 50  0001 C CNN
-	1    2050 1250
-	1    0    0    -1
-$EndComp
-Text GLabel 1100 1450 0    50   Input ~ 0
+P 550 1550
+F 0 "#PWR03" H 550 1400 50  0001 C CNN
+F 1 "+5V" H 565 1723 50  0000 C CNN
+F 2 "" H 550 1550 50  0001 C CNN
+F 3 "" H 550 1550 50  0001 C CNN
+	1    550  1550
+	1    0    0    -1
+$EndComp
+Text GLabel 1100 1350 0    50   Input ~ 0
 Audio_In_L
-Wire Wire Line
-	1100 1450 1250 1450
+Text GLabel 1900 1350 2    50   Output ~ 0
+Audio_Out_L
 Text GLabel 1900 1450 2    50   Output ~ 0
-Audio_Out_L
-Text GLabel 1900 1350 2    50   Output ~ 0
 Audio_Out_R
-Text GLabel 1100 1550 0    50   Input ~ 0
+Text GLabel 1900 1250 2    50   Input ~ 0
 Mic_In
-Wire Wire Line
-	1100 1550 1250 1550
-Text GLabel 1900 1550 2    50   Output ~ 0
+Text GLabel 1100 1250 0    50   Output ~ 0
 Mic_Out
 Wire Wire Line
@@
 Wire Wire Line
 	1750 1350 1900 1350
-NoConn ~ 1250 1350
-Wire Wire Line
-	1250 1250 950  1250
-Wire Wire Line
-	950  1250 950  1150
-Wire Wire Line
-	950  1150 800  1150
-Wire Wire Line
-	1750 1250 2050 1250
 Wire Wire Line
 	6300 1850 6650 1850
@@
 F 0 "C1" H 1815 3246 50  0000 L CNN
 F 1 "10uF" H 1815 3155 50  0000 L CNN
-F 2 "" H 1738 3050 50  0001 C CNN
+F 2 "Capacitors_SMD:C_0805_HandSoldering" H 1738 3050 50  0001 C CNN
 F 3 "~" H 1700 3200 50  0001 C CNN
 	1    1700 3200
@@
 F 0 "C2" H 2265 3246 50  0000 L CNN
 F 1 "1uF" H 2265 3155 50  0000 L CNN
-F 2 "" H 2188 3050 50  0001 C CNN
+F 2 "Capacitors_SMD:C_0805_HandSoldering" H 2188 3050 50  0001 C CNN
 F 3 "~" H 2150 3200 50  0001 C CNN
 	1    2150 3200
@@
 Text Notes 1150 700  0    50   ~ 0
 FT-891 Audio Breakout Pinout\n
-Text Notes 1150 900  0    50   Italic 10
-CHECK THIS BEFORE SUBMITTING PCB\n
 Text Notes 1200 4800 0    50   ~ 0
 Assumptions:\n- Power is provided via the radio microphone connection.  No isolation \nis provided between the radio and the audio circuitry, either out or in.
@@
 F 0 "R1" V 8193 2250 50  0000 C CNN
 F 1 "1" V 8284 2250 50  0000 C CNN
-F 2 "" V 8330 2250 50  0001 C CNN
+F 2 "Resistors_SMD:R_0805_HandSoldering" V 8330 2250 50  0001 C CNN
 F 3 "~" H 8400 2250 50  0001 C CNN
 	1    8400 2250
@@
 F 0 "R2" V 8193 2500 50  0000 C CNN
 F 1 "1" V 8284 2500 50  0000 C CNN
-F 2 "" V 8330 2500 50  0001 C CNN
+F 2 "Resistors_SMD:R_0805_HandSoldering" V 8330 2500 50  0001 C CNN
 F 3 "~" H 8400 2500 50  0001 C CNN
 	1    8400 2500
@@
 	1100 1900 1900 1900
 Text Notes 900  2100 0    50   ~ 0
-Microphone signal is unmodified in this version of the design
+Microphone signal is unmodified \nin this version of the design
+Wire Wire Line
+	1100 1350 1250 1350
+Wire Wire Line
+	1100 1250 1250 1250
+NoConn ~ 1250 1450
+Wire Wire Line
+	550  1550 1250 1550
+Wire Wire Line
+	1750 1250 1900 1250
+Wire Wire Line
+	4450 1750 5150 1750
 $EndSCHEMATC
