File: RX EQ Shield - Faceplate/RX EQ Shield - Faceplate.kicad_pcb (KiCad board)
At the start: 2 copper layers, 69.8 x 38.1 mm, 7 parts

Commit message: Faceplate ordered
Parts:
- added G***: LOGO, BVH_Logos:AB4EN_Orbitron, F.Cu at (136.5, 147.2)
